File: BoardsEAGLE/R2R_v2.1.brd (EAGLE design)
At the start: 35.9 x 83.9 mm, 36 parts, among them J1 SAMACSYS_PARTS_MTC-8810NBMLNF, Q1 BSS84, Q2 BSS84, Q3 BSS84, Q4 BSS84, Q5 BSS123, Q6 BSS123, Q7 BSS123, Q8 BSS123

Commit message: Add files via upload
Parts:
- moved LED2 2.54 mm to (3.85, 63.6)
- moved LED3 2.54 mm to (3.85, 49.6)
- moved LED4 2.54 mm to (3.85, 35.6)
- moved R11 0.95 mm to (6.38, 42.3)
- moved R4 0.64 mm to (30.5, 30.4)
Routing:
- net +3V3: track 229.7 -> 216.4 mm
- net GND: track 235.6 -> 241.9 mm
- net N$2: track 10.5 -> 14.3 mm
- net OUT: track 114.3 -> 112.3 mm
- net N$9: track 13.4 -> 11.4 mm
- net N$11: track 10.2 -> 12.1 mm
- net N$13: track 29.3 -> 27.6 mm
- net N$12: track 10.1 -> 11.7 mm
- net N$10: track 10.4 -> 11.7 mm
- net N$15: track 37.6 -> 36.7 mm
Other:
- outline, holes or cut-outs redrawn
